Commit message: Completed

File: turtlebot_description/robots/kobuki_hexagons_astra.urdf.xacro (robot description, xacro)
@@ -10,4 +10,5 @@
   <xacro:include filename="$(find turtlebot_description)/urdf/stacks/hexagons.urdf.xacro"/>
   <xacro:include filename="$(find turtlebot_description)/urdf/sensors/astra.urdf.xacro"/>
+  <link name="world"/>
   <xacro:kobuki/>
   <xacro:stack_hexagons parent="base_link"/>
