Commit message: Minor fix

File: kobuki_description/urdf/kobuki.urdf.xacro (robot description, xacro)
@@ -11,5 +11,4 @@
   <!-- Kobuki -->
   <xacro:macro name="kobuki">
-    <link name="base_footprint"/>
     <!--
        Base link is set at the bottom of the base mould.
@@ -21,9 +20,9 @@
        to 0.352.
       -->
-    <joint name="base_joint" type="fixed">
+    <!-- <joint name="base_joint" type="fixed">
       <origin xyz="0 0 0.0102" rpy="0 0 0" />
       <parent link="base_footprint"/>
       <child link="base_link" />
-    </joint>
+    </joint> -->
     <link name="base_link">
       <visual>

File: turtlebot_description/robots/kobuki_hexagons_astra.urdf.xacro (robot description, xacro)
@@ -10,7 +10,11 @@
   <xacro:include filename="$(find turtlebot_description)/urdf/stacks/hexagons.urdf.xacro"/>
   <xacro:include filename="$(find turtlebot_description)/urdf/sensors/astra.urdf.xacro"/>
-  <link name="world"/>
+  <link name="base_footprint"/>
+  <joint name="base_joint" type="fixed">
+    <parent link="base_footprint"/>
+    <child link="base_link"/>
+  </joint>
   <xacro:kobuki/>
   <xacro:stack_hexagons parent="base_link"/>
-  <xacro:sensor_astra   parent="base_link"/>
+  <xacro:sensor_astra parent="base_link"/>
 </robot>
